Commit message: add camera to simulation

File: catkin_ws/src/robocar_description/urdf/robocar.urdf (robot description, URDF)
Before this commit: robot robocar, 1 links, 0 joints
Links:
- added link camera, mass 0.1; collision box size=0.05 0.05 0.05; visual box size=0.05 0.05 0.05
Joints:
- added joint camera_joint: type fixed, parent base, child camera, origin xyz=0.2 0 ${height} rpy=0 0.2 0, axis 0 1 0
