Commit message: add camera to car model in simulation; configure rviz; a car can go straight along x axis

File: catkin_ws/src/robocar_ackermann_description/urdf/car.xacro (robot description, xacro)
@@ -271,6 +271,81 @@
   <xacro:rear_wheel lr_prefix="left" fr_prefix="rear" lr_reflect="1" fr_reflect="-1"/>
   <xacro:rear_wheel lr_prefix="right" fr_prefix="rear" lr_reflect="-1" fr_reflect="-1"/>
+  <!-- camera -->
+  <gazebo reference="camera">
+    <sensor type="camera" name="camera1">
+      <update_rate>10.0</update_rate>
+      <camera name="head">
+        <horizontal_fov>2.3</horizontal_fov>
+        <image>
+          <width>1280</width>
+          <height>960</height>
+          <format>R8G8B8</format>
+        </image>
+        <clip>
+          <near>0.02</near>
+          <far>100</far>
+        </clip>
+      </camera>
+      <plugin name="camera_controller" filename="libgazebo_ros_camera.so">
+        <alwaysOn>true</alwaysOn>
+        <updateRate>0.0</updateRate>
+        <cameraName>camera</cameraName>
+        <imageTopicName>rgb/image_raw</imageTopicName>
+        <cameraInfoTopicName>rgb/camera_info</cameraInfoTopicName>
+        <frameName>camera</frameName>
+        <hackBaseline>0.07</hackBaseline>
+        <distortionK1>-0.279653</distortionK1>
+        <distortionK2>0.060243</distortionK2>
+        <distortionK3>0.002379</distortionK3>
+        <distortionT1>-0.000038</distortionT1>
+        <distortionT2>0.0</distortionT2>
+      </plugin>
+    </sensor>
+    <material>Gazebo/Orange</material>
+  </gazebo>
+  <!-- CAMERA -->
+  <link name="camera">
+    <inertial>
+      <mass value="0.1"/>
+      <origin xyz="0 0 0" rpy=" 0 0 0"/>
+      <inertia
+          ixx="1e-6" ixy="0" ixz="0"
+          iyy="1e-6" iyz="0"
+          izz="1e-6"
+      />
+    </inertial>
+    <collision name='camera_collision'>
+      <origin xyz="0 0 0" rpy=" 0 0 0"/>
+      <geometry>
+        <box size="0.05 0.05 0.05"/>
+      </geometry>
+    </collision>
+    <visual name='camera_visual'>
+      <origin xyz="0 0 0" rpy=" 0 0 0"/>
+      <geometry>
+        <box size="0.05 0.05 0.05"/>
+      </geometry>
+    </visual>
+  </link>
+  <joint type="fixed" name="camera_joint">
+    <origin xyz="0.2 0 ${chassis_height}" rpy="0 0.2 0"/>
+    <child link="camera"/>
+    <parent link="base_link"/>
+    <axis xyz="0 1 0" rpy="0 0 0"/>
+  </joint>
+  <!-- CAMERA END -->
   <gazebo>
     <plugin name="gazebo_ros_control" filename="libgazebo_ros_control.so"/>
+    <!-- publish ground truth into odometry topic -->
+    <plugin name="p3d_base_controller" filename="libgazebo_ros_p3d.so">
+      <alwaysOn>true</alwaysOn>
+      <updateRate>50.0</updateRate>
+      <bodyName>base_link</bodyName>
+      <topicName>robocar/odometry</topicName>
+      <gaussianNoise>0.01</gaussianNoise>
+      <frameName>world</frameName>
+      <xyzOffsets>0 0 0</xyzOffsets>
+      <rpyOffsets>0 0 0</rpyOffsets>
+    </plugin>
   </gazebo>
 </robot>

Commit message: added world with straight road changed pid supervisor to use lf vector

File: catkin_ws/src/robocar_ackermann_description/urdf/car.xacro (robot description, xacro)
@@ -329,5 +329,5 @@
   </link>
   <joint type="fixed" name="camera_joint">
-    <origin xyz="0.2 0 ${chassis_height}" rpy="0 0.2 0"/>
+    <origin xyz="0.2 0 ${chassis_height+0.2}" rpy="0 0.2 0"/>
     <child link="camera"/>
     <parent link="base_link"/>

Commit message: added more nodes: - image tresholing - fitting polynomials to lane lines

File: catkin_ws/src/robocar_ackermann_description/urdf/car.xacro (robot description, xacro)
@@ -291,13 +291,17 @@
         <updateRate>0.0</updateRate>
         <cameraName>camera</cameraName>
-        <imageTopicName>rgb/image_raw</imageTopicName>
-        <cameraInfoTopicName>rgb/camera_info</cameraInfoTopicName>
+        <imageTopicName>color/image_raw</imageTopicName>
+        <cameraInfoTopicName>color/camera_info</cameraInfoTopicName>
         <frameName>camera</frameName>
-        <hackBaseline>0.07</hackBaseline>
+        <!-- 286. TODO camera matrix as in file, two numbers left-->
+        <focalLength>742.64</focalLength>
+        <CxPrime>666.99677</CxPrime>
+        <Cx>666.99677</Cx>
+        <Cy>517.3488</Cy>
         <distortionK1>-0.279653</distortionK1>
         <distortionK2>0.060243</distortionK2>
-        <distortionK3>0.002379</distortionK3>
-        <distortionT1>-0.000038</distortionT1>
-        <distortionT2>0.0</distortionT2>
+        <distortionK3>0.0</distortionK3>
+        <distortionT1>0.002379</distortionT1>
+        <distortionT2>-0.000038</distortionT2>
       </plugin>
     </sensor>
@@ -329,5 +333,5 @@
   </link>
   <joint type="fixed" name="camera_joint">
-    <origin xyz="0.2 0 ${chassis_height+0.2}" rpy="0 0.2 0"/>
+    <origin xyz="0.2 0 ${chassis_height+0.2}" rpy="0 0 0"/>
     <child link="camera"/>
     <parent link="base_link"/>

Commit message: more realistic measurements of the car

File: catkin_ws/src/robocar_ackermann_description/urdf/car.xacro (robot description, xacro)
@@ -20,17 +20,13 @@
   <!-- chassis_length is measured along the x axis, chassis_width
        along the y axis, and chassis_height along the z axis. -->
-  <xacro:property name="chassis_length" value="0.258"/>
-  <xacro:property name="chassis_width" value="0.168"/>
+  <xacro:property name="chassis_length" value="0.40"/>
+  <xacro:property name="chassis_width" value="0.15"/>
   <xacro:property name="chassis_height" value="0.01"/>
   <xacro:property name="chassis_mass" value="2.788"/>
   <!-- hub_dia and tire_dia are the diameters of the hub and tire,
-       respectively. hex_hub_depth is the distance that the hex hub is
-       inset from the outer edge of the tire. It is set so that each wheel
-       is a "zero offset" wheel. hex_hub_depth = tire_width / 2 -
-       axle_length. -->
-  <xacro:property name="hub_dia" value="0.09652"/>
-  <xacro:property name="tire_dia" value="0.14605"/>
-  <xacro:property name="tire_width" value="0.0889"/>
-  <xacro:property name="hex_hub_depth" value="0.01445"/>
+       respectively. -->
+  <xacro:property name="hub_dia" value="0.7"/>
+  <xacro:property name="tire_dia" value="0.10"/>
+  <xacro:property name="tire_width" value="0.05"/>
   <xacro:property name="wheel_mass" value="0.29"/>
   <!-- hex_hub_dist is the distance between left and right hex hubs when
@@ -38,9 +34,14 @@
        from a U joint to the corresponding hex hub. wheel_travel is the
        vertical wheel travel. -->
-  <xacro:property name="wheelbase" value="0.335"/>
-  <xacro:property name="hex_hub_dist" value="0.365"/>
+  <xacro:property name="wheelbase" value="0.30"/>
+  <xacro:property name="hex_hub_dist" value="0.33"/>
   <xacro:property name="axle_length" value="0.03"/>
   <xacro:property name="wheel_travel" value="0.084"/>
   <xacro:property name="shock_z_offset" value="0.0655"/>
+  <!-- hex_hub_depth is the distance that the hex hub is
+       inset from the outer edge of the tire. It is set so that each wheel
+       is a "zero offset" wheel. hex_hub_depth = tire_width / 2 -
+       axle_length. -->
+  <xacro:property name="hex_hub_depth" value="${tire_width / 2 - axle_length}"/>
   <!-- shock_eff_limit is 2 * ((shock_stroke / 2) * shock_spring_constant) N.
        shock_stroke is 0.028575 meters. shock_spring_constant, an approximation
@@ -311,5 +312,5 @@
   <link name="camera">
     <inertial>
-      <mass value="0.1"/>
+      <mass value="0.001"/>
       <origin xyz="0 0 0" rpy=" 0 0 0"/>
       <inertia
@@ -333,7 +334,7 @@
   </link>
   <joint type="fixed" name="camera_joint">
-    <origin xyz="0.2 0 ${chassis_height+0.2}" rpy="0 0 0"/>
+    <origin xyz="0.2 0 ${0.36}" rpy="0 ${pi / 3} 0"/>
     <child link="camera"/>
-    <parent link="base_link"/>
+    <parent link="chassis"/>
     <axis xyz="0 1 0" rpy="0 0 0"/>
   </joint>

Commit message: - transform waypoints from 'base_link' frame to the 'world' frame; - minor changes with camera pitch

File: catkin_ws/src/robocar_ackermann_description/urdf/car.xacro (robot description, xacro)
@@ -334,5 +334,5 @@
   </link>
   <joint type="fixed" name="camera_joint">
-    <origin xyz="0.2 0 ${0.36}" rpy="0 ${pi / 3} 0"/>
+    <origin xyz="0.2 0 ${0.36}" rpy="0 0 0"/>
     <child link="camera"/>
     <parent link="chassis"/>

Commit message: added optical frame for camera with Z-axis forward

File: catkin_ws/src/robocar_ackermann_description/urdf/car.xacro (robot description, xacro)
@@ -294,5 +294,6 @@
         <imageTopicName>color/image_raw</imageTopicName>
         <cameraInfoTopicName>color/camera_info</cameraInfoTopicName>
-        <frameName>camera</frameName>
+        <!-- camera frame with Z forward -->
+        <frameName>camera_link_optical</frameName>
         <!-- 286. TODO camera matrix as in file, two numbers left-->
         <focalLength>944.023585</focalLength>
@@ -327,5 +328,5 @@
     </collision>
     <visual name='camera_visual'>
-      <origin xyz="0 0 0" rpy=" 0 0 0"/>
+      <origin xyz="0 0 0" rpy="0 0 0"/>
       <geometry>
         <box size="0.05 0.05 0.05"/>
@@ -337,6 +338,19 @@
     <child link="camera"/>
     <parent link="chassis"/>
-    <axis xyz="0 1 0" rpy="0 0 0"/>
   </joint>
+  <!-- generate an optical frame
+      http://www.ros.org/reps/rep-0103.html#suffix-frames
+      so that ros and opencv can operate on the camera frame correctly
+      -->
+  <joint name="camera_optical_joint" type="fixed">
+    <!-- these values have to be these values otherwise the gazebo camera
+        image won't be aligned properly with the frame it is supposedly
+        originating from -->
+    <origin xyz="0 0 0" rpy="${-degrees_90} 0 ${-degrees_90}"/>
+    <parent link="camera"/>
+    <child link="camera_link_optical"/>
+  </joint>
+  <link name="camera_link_optical">
+  </link>
   <!-- CAMERA END -->
   <gazebo>

Commit message: added bottom_base_link

File: catkin_ws/src/robocar_ackermann_description/urdf/car.xacro (robot description, xacro)
@@ -351,4 +351,12 @@
   </link>
   <!-- CAMERA END -->
+  <!-- projection of base_link to the ground -->
+  <link name="base_bottom_link">
+  </link>
+  <joint type="fixed" name="base_to_bottom_joint">
+    <origin xyz="0 0 ${(chassis_height + wheel_travel + tire_dia) / 2}" rpy="0 0 0"/>
+    <child link="base_link"/>
+    <parent link="base_bottom_link"/>
+  </joint>
   <gazebo>
     <plugin name="gazebo_ros_control" filename="libgazebo_ros_control.so"/>
@@ -360,5 +368,5 @@
       <topicName>robocar/odometry</topicName>
       <gaussianNoise>0.01</gaussianNoise>
-      <frameName>world</frameName>
+      <frameName>base_link</frameName>
       <xyzOffsets>0 0 0</xyzOffsets>
       <rpyOffsets>0 0 0</rpyOffsets>
